Commit message: 5.23
Co-authored-by: Copilot <copilot@github.com>

File: src/arm/model/robotic_arm.urdf (robot description, URDF)
Before this commit: robot 5.142525半成品直驱机械臂装配体urdf, 8 links, 7 joints
Joints:
- joint joint1: limit lower=-1.8 upper=1.8 effort=50 velocity=10 -> lower=-3.14 upper=3.14 effort=50 velocity=10
