Commit message: 修正URDF和MJCF模型，完成测试节点，完善动作执行函数

File: src/arm/model/robotic_arm.urdf (robot description, URDF)
Before this commit: robot robotic_arm, 8 links, 7 joints
Joints:
- joint joint6: origin xyz=0.073796 0.0036822 8.8922E-05 rpy=0 -1.5708 0 -> xyz=0.073796 0.0036822 8.8922E-05 rpy=0 -1.5708 3.14

Commit message: 增加关节角限制

File: src/arm/model/robotic_arm.urdf (robot description, URDF)
Before this commit: robot robotic_arm, 8 links, 7 joints
Joints:
- joint joint1: limit lower=-6.283185307 upper=6.283185307 effort=50 velocity=10 -> lower=-1.8 upper=1.8 effort=50 velocity=10
- joint joint3: limit lower=-3.141592654 upper=3.141592654 effort=50 velocity=10 -> lower=-2.9 upper=2.9 effort=50 velocity=10
- joint joint4: limit lower=-3.141592654 upper=3.141592654 effort=50 velocity=10 -> lower=-2.0 upper=1.8 effort=50 velocity=10

Commit message: 目前面临腕关节轨迹异常

File: src/arm/model/robotic_arm.urdf (robot description, URDF)
Before this commit: robot robotic_arm, 8 links, 7 joints
Links:
- removed link link6
- link base_link: mass 1.0998 -> 0.21159
- link link1: mass 2.34956808405639 -> 0.713591271917209
- link link2: mass 1.23727124080295 -> 0.16131257849395
- link link3: mass 0.370266089775016 -> 0.0902003371394342
- link link4: mass 1.54177209165349 -> 0.0295188270468399
- link link5: mass 0.0698721570199944 -> 0.00753040773327418
Joints:
- removed joint joint6
- joint joint1: axis 0 0 1 -> 0 0 -1; limit lower=-1.8 upper=1.8 effort=50 velocity=10 -> lower=0 upper=0 effort=0 velocity=0; origin xyz=0 0 0 rpy=0 0 0 -> xyz=0 0 0.032 rpy=0 0 0
- joint joint2: limit lower=-1.570796327 upper=1.570796327 effort=50 velocity=10 -> lower=0 upper=0 effort=0 velocity=0; origin xyz=0 0.03675 0.153 rpy=1.5708 -1.5708 0 -> xyz=0.3029 -0.0175 0.0075 rpy=-1.5708 -3.14159 0
- joint joint3: axis 0 0 1 -> 0 0 -1; limit lower=-2.9 upper=2.9 effort=50 velocity=10 -> lower=0 upper=0 effort=0 velocity=0; origin xyz=0.52 0 0.08565 rpy=0 0 0 -> xyz=0.349 0.0025 0.0435 rpy=0 0 3.14159
- joint joint4: limit lower=-2.0 upper=1.8 effort=50 velocity=10 -> lower=0 upper=0 effort=0 velocity=0; origin xyz=0.436 0 0.0225 rpy=0 0 0 -> xyz=0.183 -0.03 0 rpy=0 0 -1.5708
- joint joint5: axis 0 0 1 -> 0 0 0; limit lower=-0.610865238 upper=0.610865238 effort=50 velocity=10 -> lower=-3.14 upper=3.14 effort=100 velocity=1; origin xyz=0.07761 -0.0058889 -0.03035 rpy=-1.5708 0 0 -> xyz=0.0928 0.027656 -0.026 rpy=-3.1416 0 0; type revolute -> fixed

Commit message: 4.25

File: src/arm/model/robotic_arm.urdf (robot description, URDF)
Before this commit: robot robotic_arm, 8 links, 7 joints
Joints:
- joint joint5: limit lower=-0.610865238 upper=0.610865238 effort=50 velocity=10 -> lower=-0.0349 upper=0.0349 effort=50 velocity=10

Commit message: 更换urdf

File: src/arm/model/robotic_arm.urdf (robot description, URDF)
Before this commit: robot robotic_arm, 8 links, 7 joints
Links:
- removed link link1
- removed link link2
- removed link link3
- removed link link4
- removed link link5
- removed link link6
- added link Link1, mass 2.04146059224224; collision mesh filename=package://arm/model/Link1.STL; visual mesh filename=package://arm/model/Link1.STL
- added link Link2, mass 1.39035437028225; collision mesh filename=package://arm/model/Link2.STL; visual mesh filename=package://arm/model/Link2.STL
- added link Link3, mass 0.785255181937118; collision mesh filename=package://arm/model/Link3.STL; visual mesh filename=package://arm/model/Link3.STL
- added link Link4, mass 0.372073709541278; collision mesh filename=package://arm/model/Link4.STL; visual mesh filename=package://arm/model/Link4.STL
- added link Link5, mass 0.112220070755106; collision mesh filename=package://arm/model/Link5.STL; visual mesh filename=package://arm/model/Link5.STL
- added link Link6, mass 0.150213928644987; collision mesh filename=package://arm/model/Link6.STL; visual mesh filename=package://arm/model/Link6.STL
- link base_link: mass 1.0998 -> 1.28577081829168
Joints:
- joint joint1: child link1 -> Link1; origin xyz=0 0 0 rpy=0 0 0 -> xyz=0 0 0.05075 rpy=0 0 0
- joint joint2: child link2 -> Link2; origin xyz=0 0.03675 0.153 rpy=1.5708 -1.5708 0 -> xyz=0 0.0278300000000136 0.12375000000003 rpy=-1.5707963267949 -1.57 0; parent link1 -> Link1
- joint joint3: child link3 -> Link3; origin xyz=0.52 0 0.08565 rpy=0 0 0 -> xyz=0.500000000000005 0 -0.0455028735632288 rpy=3.14159265358979 0 0; parent link2 -> Link2
- joint joint4: child link4 -> Link4; origin xyz=0.436 0 0.0225 rpy=0 0 0 -> xyz=0.509639999999998 0 0.0110471264367704 rpy=0 0 0; parent link3 -> Link3
- joint joint5: child link5 -> Link5; origin xyz=0.07761 -0.0058889 -0.03035 rpy=-1.5708 0 0 -> xyz=0.0760000000000024 0.043999999999999 0.0245500000000014 rpy=1.57 0.37 0; parent link4 -> Link4
- joint joint6: child link6 -> Link6; origin xyz=0.073796 0.0036822 8.8922E-05 rpy=0 -1.5708 3.14 -> xyz=0.0629861815027267 0.024956030127103 0.0467500000000002 rpy=1.5707963267949 -0.25158845704293 1.94803497441332; parent link5 -> Link5

Commit message: 更改joint5度关节限制

File: src/arm/model/robotic_arm.urdf (robot description, URDF)
Before this commit: robot 4.298782525半成品直驱机械臂装配体2, 8 links, 7 joints
Joints:
- joint joint5: limit lower=-0.0349 upper=0.0349 effort=50 velocity=10 -> lower=-0.5236 upper=0.5236 effort=50 velocity=10

Commit message: 5.15

File: src/arm/model/robotic_arm.urdf (robot description, URDF)
Before this commit: robot 4.298782525半成品直驱机械臂装配体2, 8 links, 7 joints
Links:
- link Link1: mass 2.04146059224224 -> 1.7349745230456
- link Link2: mass 1.39035437028225 -> 0.787811387302493
- link Link3: mass 0.785255181937118 -> 0.494884609286345
- link Link4: mass 0.372073709541278 -> 0.236644042415221
- link Link5: mass 0.112220070755106 -> 0.425979554353247
- link Link6: mass 0.150213928644987 -> 0.232464424402596
- link base_link: mass 1.28577081829168 -> 1.01281835096414
Joints:
- joint joint1: axis 0 0 1 -> 0 0 -1; origin xyz=0 0 0.05075 rpy=0 0 0 -> xyz=0 0 0.0525 rpy=0 0 -1.5708
- joint joint2: axis 0 0 1 -> 0 0 -1; limit lower=-1.570796327 upper=1.570796327 effort=50 velocity=10 -> lower=-1.57 upper=1.57 effort=50 velocity=10; origin xyz=0 0.0278300000000136 0.12375000000003 rpy=-1.5707963267949 -1.57 0 -> xyz=0 0.02652 0.122 rpy=1.5708 -1.57 0
- joint joint3: axis 0 0 1 -> 0 0 -1; origin xyz=0.500000000000005 0 -0.0455028735632288 rpy=3.14159265358979 0 0 -> xyz=0.5 0 0.0445 rpy=0 0 0
- joint joint4: axis 0 0 1 -> 0 0 -1; origin xyz=0.509639999999998 0 0.0110471264367704 rpy=0 0 0 -> xyz=0.47447 0 0.0085 rpy=-3.1416 0 0
- joint joint5: axis 0 0 1 -> 0 0 -1; origin xyz=0.0760000000000024 0.043999999999999 0.0245500000000014 rpy=1.57 0.37 0 -> xyz=0.076 -0.0435 -0.02685 rpy=1.57 -0.37 0
- joint joint6: limit lower=-3.14159 upper=3.14159 effort=50 velocity=10 -> lower=-0.01 upper=0.01 effort=50 velocity=10; origin xyz=0.0629861815027267 0.024956030127103 0.0467500000000002 rpy=1.5707963267949 -0.25158845704293 1.94803497441332 -> xyz=0.079534 -0.016991 -0.02705 rpy=0 0 -0.37724

Commit message: old model

File: src/arm/model/robotic_arm.urdf (robot description, URDF)
Before this commit: robot 4.298782525半成品直驱机械臂装配体2, 8 links, 7 joints
Links:
- removed link Link1
- removed link Link2
- removed link Link3
- removed link Link4
- removed link Link5
- removed link Link6
- added link link1, mass 2.34956808405639; collision mesh filename=package://arm/model/link1.STL; visual mesh filename=package://arm/model/link1.STL
- added link link2, mass 1.23727124080295; collision mesh filename=package://arm/model/link2.STL; visual mesh filename=package://arm/model/link2.STL
- added link link3, mass 0.370266089775016; collision mesh filename=package://arm/model/link3.STL; visual mesh filename=package://arm/model/link3.STL
- added link link4, mass 1.54177209165349; collision mesh filename=package://arm/model/link4.STL; visual mesh filename=package://arm/model/link4.STL
- added link link5, mass 0.0698721570199944; collision mesh filename=package://arm/model/link5.STL; visual mesh filename=package://arm/model/link5.STL
- added link link6, mass 0.128099358994803; collision mesh filename=package://arm/model/link6.STL; visual mesh filename=package://arm/model/link6.STL
- link base_link: mass 1.28577081829168 -> 1.0998
Joints:
- joint joint1: child Link1 -> link1; origin xyz=0 0 0.05075 rpy=0 0 0 -> xyz=0 0 0 rpy=0 0 0
- joint joint2: child Link2 -> link2; origin xyz=0 0.0278300000000136 0.12375000000003 rpy=-1.5707963267949 -1.57 0 -> xyz=0 0.03675 0.153 rpy=1.5708 -1.5708 0; parent Link1 -> link1
- joint joint3: child Link3 -> link3; origin xyz=0.500000000000005 0 -0.0455028735632288 rpy=3.14159265358979 0 0 -> xyz=0.52 0 0.08565 rpy=0 0 -0.35; parent Link2 -> link2
- joint joint4: child Link4 -> link4; origin xyz=0.509639999999998 0 0.0110471264367704 rpy=0 0 0 -> xyz=0.436 0 0.0225 rpy=0 0 0; parent Link3 -> link3
- joint joint5: child Link5 -> link5; limit lower=-0.5236 upper=0.5236 effort=50 velocity=10 -> lower=-0.0349 upper=0.0349 effort=50 velocity=10; origin xyz=0.0760000000000024 0.043999999999999 0.0245500000000014 rpy=1.57 0.37 0 -> xyz=0.07761 -0.0058889 -0.03035 rpy=-1.5708 0 0; parent Link4 -> link4
- joint joint6: child Link6 -> link6; origin xyz=0.0629861815027267 0.024956030127103 0.0467500000000002 rpy=1.5707963267949 -0.25158845704293 1.94803497441332 -> xyz=0.073796 0.0036822 8.8922E-05 rpy=0 -1.5708 3.14; parent Link5 -> link5

Commit message: 直接读末端位置

File: src/arm/model/robotic_arm.urdf (robot description, URDF)
Before this commit: robot 5.142525半成品直驱机械臂装配体urdf, 8 links, 7 joints
Joints:
- joint joint1: axis 0 0 -1 -> 0 0 1

Commit message: 跟换模型

File: src/arm/model/robotic_arm.urdf (robot description, URDF)
Before this commit: robot 5.142525半成品直驱机械臂装配体urdf, 8 links, 7 joints
Links:
- added link Link7, mass 0.23387; collision mesh filename=package://arm/model/Link7.STL; visual mesh filename=package://arm/model/Link7.STL
- link Link1: mass 1.7349745230456 -> 1.7203
- link Link2: mass 0.787811387302493 -> 0.78781
- link Link3: mass 0.494884609286345 -> 0.49488
- link Link4: mass 0.236644042415221 -> 0.23664
- link Link5: mass 0.425979554353247 -> 0.40058
- link Link6: mass 0.232464424402596 -> 0.0254009547015186
- link base_link: mass 1.01281835096414 -> 1.0128
Joints:
- added joint joint7: type fixed, parent Link6, child Link7, origin xyz=0.0075 0.0015 0.06595 rpy=0 -1.5708 0, axis 0 0 0
- joint joint1: origin xyz=0 0 0.0525 rpy=0 0 -1.5708 -> xyz=0 0 0.0525 rpy=0 0 0
- joint joint2: origin xyz=0 0.02652 0.122 rpy=1.5708 -1.57 0 -> xyz=0 0.02652 0.122 rpy=1.5708 -1.5708 0
- joint joint4: limit lower=-2.0 upper=1.8 effort=50 velocity=10 -> lower=-2.0 upper=1.3 effort=50 velocity=10; origin xyz=0.47447 0 0.0085 rpy=-3.1416 0 0 -> xyz=0.50964 0 0.0085 rpy=-3.141 0 0
- joint joint5: limit lower=-0.5236 upper=0.5236 effort=50 velocity=10 -> lower=-0.43 upper=0.43 effort=50 velocity=10; origin xyz=0.076 -0.0435 -0.02685 rpy=1.57 -0.37 0 -> xyz=0.072118 -0.049671 -0.02685 rpy=1.5708 -0.34 0
- joint joint6: limit lower=-0.01 upper=0.01 effort=50 velocity=10 -> lower=-1 upper=1 effort=50 velocity=10; origin xyz=0.079534 -0.016991 -0.02705 rpy=0 0 -0.37724 -> xyz=0.048576 -0.019247 -0.04625 rpy=0.377 -1.5708 2.415

Commit message: 5.28

File: src/arm/model/robotic_arm.urdf (robot description, URDF)
Before this commit: robot 5.142525半成品直驱机械臂装配体urdf夹爪, 9 links, 8 joints
Links:
- added link end_effector, mass 0.001; visual sphere radius=0.015
Joints:
- added joint joint8: type fixed, parent Link7, child end_effector, origin xyz=0 0 0.02 rpy=0 0 0, axis 0 0 0

Commit message: 5.31

File: src/arm/model/robotic_arm.urdf (robot description, URDF)
Before this commit: robot 5.142525半成品直驱机械臂装配体urdf夹爪, 10 links, 9 joints
Links:
- removed link end_effector
- link Link1: mass 1.7203 -> 1.72029055581718
- link Link2: mass 0.78781 -> 0.787811387302494
- link Link3: mass 0.49488 -> 0.494884613006494
- link Link4: mass 0.23664 -> 0.236643991494003
- link Link5: mass 0.40058 -> 0.243627744303709
- link Link7: mass 0.23387 -> 0.233866731874561
- link base_link: mass 1.0128 -> 1.01281835096414
Joints:
- removed joint joint8
- joint joint1: axis 0 0 1 -> 0 0 -1; limit lower=-3.14 upper=3.14 effort=50 velocity=10 -> lower=-3 upper=3 effort=50 velocity=10; origin xyz=0 0 0.0525 rpy=0 0 0 -> xyz=0 0 0.0524999999999884 rpy=0 0 0
- joint joint2: origin xyz=0 0.02652 0.122 rpy=1.5708 -1.5708 0 -> xyz=0 0.0265199999999967 0.122000000000151 rpy=1.5707963267949 -1.5708 0
- joint joint3: limit lower=-2.9 upper=2.9 effort=50 velocity=10 -> lower=-3 upper=3 effort=50 velocity=10; origin xyz=0.5 0 0.0445 rpy=0 0 0 -> xyz=0.500000000000009 0 0.0445000000000004 rpy=0 0 0
- joint joint4: limit lower=-2.0 upper=1.3 effort=50 velocity=10 -> lower=-2.5 upper=1.3 effort=50 velocity=10; origin xyz=0.50964 0 0.0085 rpy=-3.141 0 0 -> xyz=0.509641016151201 0 0.00849999999999872 rpy=-3.1415926535897 0 0
- joint joint5: axis 0 0 -1 -> 0 0 1; limit lower=-0.43 upper=0.43 effort=50 velocity=10 -> lower=-0.4 upper=0.4 effort=50 velocity=10; origin xyz=0.072118 -0.049671 -0.02685 rpy=1.5708 -0.34 0 -> xyz=0.0721180192043501 -0.0496713328390738 -0.0268500000004852 rpy=-1.5707963267949 0.0 0.0
- joint joint6: limit lower=-1 upper=1 effort=50 velocity=10 -> lower=-0.1 upper=0.1 effort=50 velocity=10; origin xyz=0.048576 -0.019247 -0.04625 rpy=0.377 -1.5708 2.415 -> xyz=0.0522500000000078 0 0.0462500000000007 rpy=0.0 1.57079631189374 0.0
- joint joint7: origin xyz=0.0075 0.0015 0.06595 rpy=0 -1.5708 0 -> xyz=0.00749999999999929 0.00150000000000178 0.0659500000000004 rpy=2.01799595197509 -1.57079631189374 1.11206808047685

Commit message: new urdf

File: src/arm/model/robotic_arm.urdf (robot description, URDF)
Before this commit: robot 5.142525半成品直驱机械臂装配体78989789urdfxin, 9 links, 8 joints
Links:
- removed link Link7
- link Link1: mass 1.72029055581718 -> 1.3415964916658
- link Link2: mass 0.787811387302494 -> 1.1688360536306
- link Link3: mass 0.494884613006494 -> 0.697933163337346
- link Link4: mass 0.236643991494003 -> 0.37892648177412
- link Link5: mass 0.243627744303709 -> 0.112337074738347
- link Link6: mass 0.0254009547015186 -> 0.150213928644986
- link base_link: mass 1.01281835096414 -> 1.0608896790749
Joints:
- removed joint joint7
- joint joint1: limit lower=-3 upper=3 effort=50 velocity=10 -> lower=-2.1 upper=2.1 effort=50 velocity=10; origin xyz=0 0 0.0524999999999884 rpy=0 0 0 -> xyz=0 0 0.04875 rpy=0 0 0
- joint joint2: origin xyz=0 0.0265199999999967 0.122000000000151 rpy=1.5707963267949 -1.5708 0 -> xyz=0 -0.02575 0.08875 rpy=-1.5708 -1.5708 0
- joint joint3: axis 0 0 -1 -> 0 0 1; limit lower=-3 upper=3 effort=50 velocity=10 -> lower=-2.9 upper=2.9 effort=50 velocity=10; origin xyz=0.500000000000009 0 0.0445000000000004 rpy=0 0 0 -> xyz=0.5 0 0.044 rpy=0 0 0
- joint joint4: limit lower=-2.5 upper=1.3 effort=50 velocity=10 -> lower=-2 upper=2 effort=50 velocity=10; origin xyz=0.509641016151201 0 0.00849999999999872 rpy=-3.1415926535897 0 0 -> xyz=0.49464 0 0.04645 rpy=0 0 0
- joint joint5: axis 0 0 1 -> 0 0 -1; origin xyz=0.0721180192043501 -0.0496713328390738 -0.0268500000004852 rpy=-1.5707963267949 0.0 0.0 -> xyz=0.076 -0.044 -0.02455 rpy=-1.5708 0 0
- joint joint6: limit lower=-0.1 upper=0.1 effort=50 velocity=10 -> lower=0 upper=0 effort=50 velocity=10; origin xyz=0.0522500000000078 0 0.0462500000000007 rpy=0.0 1.57079631189374 0.0 -> xyz=0.055 0 0.04675 rpy=-1.333 1.5708 -1.4022

Commit message: 6.23

File: src/arm/model/robotic_arm.urdf (robot description, URDF)
Before this commit: robot 5.142525半成品直驱机械臂装配体78989789urdfxin, 9 links, 8 joints
Links:
- removed link Link1
- removed link Link2
- removed link Link3
- removed link Link4
- removed link Link5
- removed link Link6
- removed link Link7
- added link link1, mass 1.3415964916658; collision mesh filename=package://arm/model/Link1.STL; visual mesh filename=package://arm/model/Link1.STL
- added link link2, mass 1.1688360536306; collision mesh filename=package://arm/model/Link2.STL; visual mesh filename=package://arm/model/Link2.STL
- added link link3, mass 0.697933163337346; collision mesh filename=package://arm/model/Link3.STL; visual mesh filename=package://arm/model/Link3.STL
- added link link4, mass 0.37892648177412; collision mesh filename=package://arm/model/Link4.STL; visual mesh filename=package://arm/model/Link4.STL
- added link link5, mass 0.112337074738347; collision mesh filename=package://arm/model/Link5.STL; visual mesh filename=package://arm/model/Link5.STL
- added link link6, mass 0.150213928644986; collision mesh filename=package://arm/model/Link6.STL; visual mesh filename=package://arm/model/Link6.STL
- link base_link: mass 1.01281835096414 -> 1.0608896790749
Joints:
- removed joint joint7
- joint joint1: child Link1 -> link1; limit lower=-3 upper=3 effort=50 velocity=10 -> lower=-2.1 upper=2.1 effort=50 velocity=10; origin xyz=0 0 0.0524999999999884 rpy=0 0 0 -> xyz=0 0 0.04875 rpy=0 0 0
- joint joint2: child Link2 -> link2; origin xyz=0 0.0265199999999967 0.122000000000151 rpy=1.5707963267949 -1.5708 0 -> xyz=0 -0.02575 0.08875 rpy=-1.5708 -1.5708 0; parent Link1 -> link1
- joint joint3: axis 0 0 -1 -> 0 0 1; child Link3 -> link3; limit lower=-3 upper=3 effort=50 velocity=10 -> lower=-2.9 upper=2.9 effort=50 velocity=10; origin xyz=0.500000000000009 0 0.0445000000000004 rpy=0 0 0 -> xyz=0.5 0 0.044 rpy=0 0 0; parent Link2 -> link2
- joint joint4: child Link4 -> link4; limit lower=-2.5 upper=1.3 effort=50 velocity=10 -> lower=-2 upper=2 effort=50 velocity=10; origin xyz=0.509641016151201 0 0.00849999999999872 rpy=-3.1415926535897 0 0 -> xyz=0.49464 0 0.04645 rpy=0 0 0; parent Link3 -> link3
- joint joint5: axis 0 0 1 -> 0 0 -1; child Link5 -> link5; origin xyz=0.0721180192043501 -0.0496713328390738 -0.0268500000004852 rpy=-1.5707963267949 0.0 0.0 -> xyz=0.076 -0.044 -0.02455 rpy=-1.5708 0 0; parent Link4 -> link4
- joint joint6: child Link6 -> link6; limit lower=-0.1 upper=0.1 effort=50 velocity=10 -> lower=0 upper=0 effort=50 velocity=10; origin xyz=0.0522500000000078 0 0.0462500000000007 rpy=0.0 1.57079631189374 0.0 -> xyz=0.055 0 0.04675 rpy=-1.333 1.5708 -1.4022; parent Link5 -> link5

Commit message: 修复urdf和项目文件不匹配的问题。

File: src/arm/model/robotic_arm.urdf (robot description, URDF)
Before this commit: robot 质修R2仿制电科云台机械臂666URDF, 8 links, 7 joints
Links:
- removed link link1
- removed link link2
- removed link link3
- removed link link4
- removed link link5
- removed link link6
- added link Link1, mass 1.3415964916658; collision mesh filename=package://arm/model/Link1.STL; visual mesh filename=package://arm/model/Link1.STL
- added link Link2, mass 1.1688360536306; collision mesh filename=package://arm/model/Link2.STL; visual mesh filename=package://arm/model/Link2.STL
- added link Link3, mass 0.697933163337346; collision mesh filename=package://arm/model/Link3.STL; visual mesh filename=package://arm/model/Link3.STL
- added link Link4, mass 0.37892648177412; collision mesh filename=package://arm/model/Link4.STL; visual mesh filename=package://arm/model/Link4.STL
- added link Link5, mass 0.112337074738347; collision mesh filename=package://arm/model/Link5.STL; visual mesh filename=package://arm/model/Link5.STL
- added link Link6, mass 0.150213928644986; collision mesh filename=package://arm/model/Link6.STL; visual mesh filename=package://arm/model/Link6.STL
Joints:
- joint joint1: child link1 -> Link1
- joint joint2: child link2 -> Link2; parent link1 -> Link1
- joint joint3: child link3 -> Link3; parent link2 -> Link2
- joint joint4: child link4 -> Link4; parent link3 -> Link3
- joint joint5: child link5 -> Link5; parent link4 -> Link4
- joint joint6: child link6 -> Link6; parent link5 -> Link5
