Commit message: 导入了新的机械臂的模型，但是目前代码框架和思路还没有

File: src/arm/model/arm4.urdf (robot description, URDF)
Before this commit: robot arm, 6 links, 5 joints
Links:
- removed link link1
- removed link link2
- removed link link3
- removed link link4
- removed link link5
- added link left1, mass 0.105541043988117; collision mesh filename=package://arm/model/left1.STL; visual mesh filename=package://arm/model/left1.STL
- added link left2, mass 0.0594508258557591; collision mesh filename=package://arm/model/left2.STL; visual mesh filename=package://arm/model/left2.STL
- added link left3, mass 0.0717898152307374; collision mesh filename=package://arm/model/left3.STL; visual mesh filename=package://arm/model/left3.STL
- added link left4, mass 0.098687873771068; collision mesh filename=package://arm/model/left4.STL; visual mesh filename=package://arm/model/left4.STL
- added link right1, mass 0.0611657666488922; collision mesh filename=package://arm/model/right1.STL; visual mesh filename=package://arm/model/right1.STL
- added link right2, mass 0.059450825942565; collision mesh filename=package://arm/model/right2.STL; visual mesh filename=package://arm/model/right2.STL
- added link right3, mass 0.0710392896004507; collision mesh filename=package://arm/model/right3.STL; visual mesh filename=package://arm/model/right3.STL
- added link right4, mass 0.0986878737710681; collision mesh filename=package://arm/model/right4.STL; visual mesh filename=package://arm/model/right4.STL
- added link yuntai, mass 0.0350606384576612; collision mesh filename=package://arm/model/yuntai.STL; visual mesh filename=package://arm/model/yuntai.STL
- link base_link: mass 0.013404874825587 -> 0.066822750433732
Joints:
- removed joint joint1
- removed joint joint2
- removed joint joint3
- removed joint joint4
- removed joint joint5
- added joint left1: type revolute, parent yuntai, child left1, origin xyz=-0.165 0.00625 0.01 rpy=1.5708 0 0, axis 0 0 -1, limit lower=0 upper=0 effort=0 velocity=0
- added joint left2: type revolute, parent left1, child left2, origin xyz=0.14795 0.02 0.00935 rpy=0 0 -3.1416, axis 0 0 1, limit lower=0 upper=0 effort=0 velocity=0
- added joint left3: type revolute, parent left2, child left3, origin xyz=0.213 0 0.0229 rpy=0 0 1.5708, axis 0 0 -1, limit lower=0 upper=0 effort=0 velocity=0
- added joint left4: type continuous, parent left3, child left4, origin xyz=0.1058 0.0275 -0.026 rpy=1.5708 0 0, axis 1 0 0
- added joint right1: type revolute, parent yuntai, child right1, origin xyz=0.165 -0.00625 0.01 rpy=1.5708 0 3.1416, axis 0 0 -1, limit lower=0 upper=0 effort=0 velocity=0
- added joint right2: type revolute, parent right1, child right2, origin xyz=0.14795 0.02 0.00935 rpy=-3.1416 0 -3.1416, axis 0 0 -1, limit lower=0 upper=0 effort=0 velocity=0
- added joint right3: type revolute, parent right2, child right3, origin xyz=0.213 0 -0.0229 rpy=0 0 -1.5708, axis 0 0 1, limit lower=0 upper=0 effort=0 velocity=0
- added joint right4: type continuous, parent right3, child right4, origin xyz=0.1058 -0.0275 0.026 rpy=-1.5708 0 0, axis 1 0 0
- added joint yuntai: type revolute, parent base_link, child yuntai, origin xyz=0 0 0.0565 rpy=0 0 0, axis 0 1 0, limit lower=0 upper=0 effort=0 velocity=0

Commit message: 当强代码在rviz2中云台旋转轴选错

File: src/arm/model/arm4.urdf (robot description, URDF)
Before this commit: robot 05双端机械臂.SLDASM, 10 links, 9 joints
Joints:
- joint left1: axis 0 0 -1 -> 0 0 1
- joint left2: axis 0 0 1 -> 0 0 -1
- joint left3: axis 0 0 -1 -> 0 0 1

Commit message: 当前模型导入有问题

File: src/arm/model/arm4.urdf (robot description, URDF)
Before this commit: robot arm, 10 links, 9 joints
Joints:
- joint left3: axis 0 0 1 -> 0 0 -1
- joint yuntai: axis 0 1 0 -> 0 0 1

Commit message: 改好的模型

File: src/arm/model/arm4.urdf (robot description, URDF)
Before this commit: robot arm, 10 links, 9 joints
Links:
- link left1: mass 0.105541043988117 -> 0.0724494118638427
- link right1: mass 0.0611657666488922 -> 0.0724494118638428
- link right4: mass 0.0986878737710681 -> 0.098687873771068
- link yuntai: mass 0.0350606384576612 -> 0.10124390270621
Joints:
- joint left4: axis 1 0 0 -> 0 0 0; type continuous -> fixed
- joint right1: axis 0 0 -1 -> 0 0 1
- joint right2: axis 0 0 -1 -> 0 0 1
- joint right4: axis 1 0 0 -> 0 -0.693904698830335 -0.720066850327927; origin xyz=0.1058 -0.0275 0.026 rpy=-1.5708 0 0 -> xyz=0.1058 -0.0274999999999999 0.0260000000000004 rpy=-1.5707963267949 0 0; type continuous -> fixed
- joint yuntai: axis 0 0 1 -> 0 0 -1

Commit message: 当前代码的笛卡尔解算无法使用，我怀疑我改废了

File: src/arm/model/arm4.urdf (robot description, URDF)
Before this commit: robot arm, 10 links, 9 joints
Joints:
- joint left4: origin xyz=0.1058 0.0275 -0.026 rpy=1.5708 0 0 -> xyz=0.1058 0.0275 -0.026 rpy=3.1416 0 0

Commit message: 非核心功能包重构

File: src/arm/model/arm4.urdf (robot description, URDF)
Before this commit: robot arm, 10 links, 9 joints
Links:
- link base_link: geometry collision mesh filename=base_link.STL; visual mesh filename=base_link.STL
- link left1: geometry collision mesh filename=left1.STL; visual mesh filename=left1.STL
- link left2: geometry collision mesh filename=left2.STL; visual mesh filename=left2.STL
- link left3: geometry collision mesh filename=left3.STL; visual mesh filename=left3.STL
- link left4: geometry collision mesh filename=left4.STL; visual mesh filename=left4.STL
- link right1: geometry collision mesh filename=right1.STL; visual mesh filename=right1.STL
- link right2: geometry collision mesh filename=right2.STL; visual mesh filename=right2.STL
- link right3: geometry collision mesh filename=right3.STL; visual mesh filename=right3.STL
- link right4: geometry collision mesh filename=right4.STL; visual mesh filename=right4.STL
- link yuntai: geometry collision mesh filename=yuntai.STL; visual mesh filename=yuntai.STL
Joints:
- joint left1: limit lower=0 upper=0 effort=0 velocity=0 -> lower=-3.14159 upper=3.14159 effort=10 velocity=10
- joint left2: limit lower=0 upper=0 effort=0 velocity=0 -> lower=-3.14159 upper=3.14159 effort=10 velocity=10
- joint left3: limit lower=0 upper=0 effort=0 velocity=0 -> lower=-3.14159 upper=3.14159 effort=10 velocity=10
- joint right1: limit lower=0 upper=0 effort=0 velocity=0 -> lower=-3.14159 upper=3.14159 effort=10 velocity=10
- joint right2: limit lower=0 upper=0 effort=0 velocity=0 -> lower=-3.14159 upper=3.14159 effort=10 velocity=10
- joint right3: limit lower=0 upper=0 effort=0 velocity=0 -> lower=-3.14159 upper=3.14159 effort=10 velocity=10
- joint yuntai: limit lower=0 upper=0 effort=0 velocity=0 -> lower=-3.14159 upper=3.14159 effort=10 velocity=10

Commit message: 调试用

File: src/arm/model/arm4.urdf (robot description, URDF)
Before this commit: robot arm, 10 links, 9 joints
Links:
- link base_link: geometry collision mesh filename=package://arm/model/base_link.STL; visual mesh filename=package://arm/model/base_link.STL
- link left1: geometry collision mesh filename=package://arm/model/left1.STL; visual mesh filename=package://arm/model/left1.STL
- link left2: geometry collision mesh filename=package://arm/model/left2.STL; visual mesh filename=package://arm/model/left2.STL
- link left3: geometry collision mesh filename=package://arm/model/left3.STL; visual mesh filename=package://arm/model/left3.STL
- link left4: geometry collision mesh filename=package://arm/model/left4.STL; visual mesh filename=package://arm/model/left4.STL
- link right1: geometry collision mesh filename=package://arm/model/right1.STL; visual mesh filename=package://arm/model/right1.STL
- link right2: geometry collision mesh filename=package://arm/model/right2.STL; visual mesh filename=package://arm/model/right2.STL
- link right3: geometry collision mesh filename=package://arm/model/right3.STL; visual mesh filename=package://arm/model/right3.STL
- link right4: geometry collision mesh filename=package://arm/model/right4.STL; visual mesh filename=package://arm/model/right4.STL
- link yuntai: geometry collision mesh filename=package://arm/model/yuntai.STL; visual mesh filename=package://arm/model/yuntai.STL

Commit message: 对坐标轴进行了修改

File: src/arm/model/arm4.urdf (robot description, URDF)
Before this commit: robot arm, 10 links, 9 joints
Joints:
- joint left1: limit lower=-3.14159 upper=3.14159 effort=10 velocity=10 -> lower=0 upper=0 effort=0 velocity=0
- joint left2: limit lower=-3.14159 upper=3.14159 effort=10 velocity=10 -> lower=0 upper=0 effort=0 velocity=0
- joint left3: limit lower=-3.14159 upper=3.14159 effort=10 velocity=10 -> lower=0 upper=0 effort=0 velocity=0
- joint left4: origin xyz=0.1058 0.0275 -0.026 rpy=3.1416 0 0 -> xyz=0.1058 0.0275 -0.026 rpy=0 0 0
- joint right1: limit lower=-3.14159 upper=3.14159 effort=10 velocity=10 -> lower=0 upper=0 effort=0 velocity=0
- joint right2: limit lower=-3.14159 upper=3.14159 effort=10 velocity=10 -> lower=0 upper=0 effort=0 velocity=0
- joint right3: limit lower=-3.14159 upper=3.14159 effort=10 velocity=10 -> lower=0 upper=0 effort=0 velocity=0
- joint right4: origin xyz=0.1058 -0.0274999999999999 0.0260000000000004 rpy=-1.5707963267949 0 0 -> xyz=0.1058 -0.0274999999999999 0.0260000000000004 rpy=0 0 0
- joint yuntai: limit lower=-3.14159 upper=3.14159 effort=10 velocity=10 -> lower=0 upper=0 effort=0 velocity=0
